File: MatrixLed/MatrixLed.sch (KiCad schematic (older format))
At the start: 76 parts, among them P1 CONN_01X04, U1 HT16K33

Commit message: Añadida serigrafia reflectante
Parts:
- C1: footprint (none) -> Capacitors_SMD:C_1206
- D1, D10, D11, D12, D13, D14, D15, D16, D17, D18, D19, D2, D20, D21, D22, D23, D24, D25, D26, D27, D28, D29, D3, D30, D31, D32, D33, D34, D35, D36, D37, D38, D39, D4, D40, D41, D42, D43, D44, D45, D46, D47, D48, D49, D5, D50, D51, D52, D53, D54, D55, D56, D57, D58, D59, D6, D60, D61, D62, D63, D64, D7, D8, D9: footprint (none) -> LEDs:LED_0603
- D65: footprint Diodes_ThroughHole:D_DO-35_SOD27_Horizontal_RM10 -> Diodes_SMD:D_SOD-123
- JP1, JP2, JP3, R1, R2, R3, R4, R5: footprint (none) -> Resistors_SMD:R_0805
- P1: footprint (none) -> Connectors_JST:JST_PH_S4B-PH-SM4-TB_04x2.00mm_Angled
- U1: footprint MODULE -> Housings_SOIC:SOIC-28W_7.5x17.9mm_Pitch1.27mm
Connections:
- net A0 renamed SEGC
- net A1 renamed SEGB
- net A2 renamed SEGA
