File: MatrixLed.kicad_pcb (KiCad board)
At the start: 2 copper layers, 58.3 x 30.4 mm, 144 parts, among them P1 CONN_01X04, U1 HT16K33

Commit message: arbol de carpetas cambiado
Parts:
- removed the G*** at (191.3, 71.0)
- added G***: LOGO, Grape:atom_small, B.Cu at (211.7, 70.7)
Other:
- board text added: "GND"
- board text added: "SCL"
- board text added: "SDA"
- board text added: "VCC"
